File: ATSAMD51_setup.sch (KiCad schematic (older format))
At the start: 24 parts, among them J2 SWD CONNECTOR, SW1 Reset_Btn, U2 ATSAMD51J19A, U3 S25FL064LABMFI013, Y1 32.768kHz

Commit message: update
Connections:
- net MISO renamed CIPO
- net MOSI renamed COPI
Other:
- note added: "heavily inspired by Adafruit M4 \nhttps://learn.adafruit.com/adafruit-metro-m4-express-featuring-atsamd51/downloads"
Changed lines of the file:
@@
 $Descr A4 11693 8268
 encoding utf-8
-Sheet 93 93
-Title ""
-Date ""
-Rev ""
+Sheet 94 94
+Title "Basic setup for ATSAMD51"
+Date "2020-08-24"
+Rev "XA2020"
 Comp ""
 Comment1 ""
 Comment2 ""
 Comment3 ""
-Comment4 ""
+Comment4 "Author: Caden Keese"
 $EndDescr
 $Comp
@@
 AR Path="/5F1F1050/5F202650" Ref="R7"  Part="1"
 AR Path="/5F45D3C3/5F202650" Ref="R7"  Part="1"
+AR Path="/5F4B2714/5F202650" Ref="R?"  Part="1"
+AR Path="/5F4B67F1/5F202650" Ref="R?"  Part="1"
+AR Path="/5F4B8821/5F202650" Ref="R?"  Part="1"
 F 0 "R7" H 1957 1204 50  0000 R CNN
 F 1 "10k" H 1957 1295 50  0000 R CNN
@@
 AR Path="/5F1F1050/5F2167CC" Ref="SW1"  Part="1"
 AR Path="/5F45D3C3/5F2167CC" Ref="SW1"  Part="1"
+AR Path="/5F4B2714/5F2167CC" Ref="SW?"  Part="1"
+AR Path="/5F4B67F1/5F2167CC" Ref="SW?"  Part="1"
+AR Path="/5F4B8821/5F2167CC" Ref="SW?"  Part="1"
 F 0 "SW1" V 1254 1998 50  0000 L CNN
 F 1 "Reset_Btn" V 1345 1998 50  0000 L CNN
@@
 AR Path="/5F1F1050/5F218D29" Ref="L1"  Part="1"
 AR Path="/5F45D3C3/5F218D29" Ref="L1"  Part="1"
+AR Path="/5F4B2714/5F218D29" Ref="L?"  Part="1"
+AR Path="/5F4B67F1/5F218D29" Ref="L?"  Part="1"
+AR Path="/5F4B8821/5F218D29" Ref="L?"  Part="1"
 F 0 "L1" V 1769 2650 50  0000 C CNN
 F 1 "10µH" V 1860 2650 50  0000 C CNN
@@
 AR Path="/5F1F1050/5F21B607" Ref="C92"  Part="1"
 AR Path="/5F45D3C3/5F21B607" Ref="C94"  Part="1"
+AR Path="/5F4B2714/5F21B607" Ref="C?"  Part="1"
+AR Path="/5F4B67F1/5F21B607" Ref="C?"  Part="1"
+AR Path="/5F4B8821/5F21B607" Ref="C?"  Part="1"
 F 0 "C94" H 1842 2921 50  0000 L CNN
 F 1 "10µF" H 1842 2830 50  0000 L CNN
@@
 AR Path="/5F1F1050/5F21A7F6" Ref="C91"  Part="1"
 AR Path="/5F45D3C3/5F21A7F6" Ref="C93"  Part="1"
+AR Path="/5F4B2714/5F21A7F6" Ref="C?"  Part="1"
+AR Path="/5F4B67F1/5F21A7F6" Ref="C?"  Part="1"
+AR Path="/5F4B8821/5F21A7F6" Ref="C?"  Part="1"
 F 0 "C93" H 1492 2921 50  0000 L CNN
 F 1 "1µF" H 1492 2830 50  0000 L CNN
@@
 AR Path="/5F1F1050/5F201B38" Ref="C89"  Part="1"
 AR Path="/5F45D3C3/5F201B38" Ref="C90"  Part="1"
+AR Path="/5F4B2714/5F201B38" Ref="C?"  Part="1"
+AR Path="/5F4B67F1/5F201B38" Ref="C?"  Part="1"
+AR Path="/5F4B8821/5F201B38" Ref="C?"  Part="1"
 F 0 "C90" H 1117 1871 50  0000 L CNN
 F 1 "1µF" H 1117 1780 50  0000 L CNN
@@
 AR Path="/5F1F1050/5F269BE6" Ref="Y1"  Part="1"
 AR Path="/5F45D3C3/5F269BE6" Ref="Y1"  Part="1"
+AR Path="/5F4B2714/5F269BE6" Ref="Y?"  Part="1"
+AR Path="/5F4B67F1/5F269BE6" Ref="Y?"  Part="1"
+AR Path="/5F4B8821/5F269BE6" Ref="Y?"  Part="1"
 F 0 "Y1" V 5454 1088 50  0000 L CNN
 F 1 "32.768kHz" V 5545 1088 50  0000 L CNN
@@
 AR Path="/5F1F1050/5F26A686" Ref="C84"  Part="1"
 AR Path="/5F45D3C3/5F26A686" Ref="C84"  Part="1"
+AR Path="/5F4B2714/5F26A686" Ref="C?"  Part="1"
+AR Path="/5F4B67F1/5F26A686" Ref="C?"  Part="1"
+AR Path="/5F4B8821/5F26A686" Ref="C?"  Part="1"
 F 0 "C84" V 5021 825 50  0000 C CNN
 F 1 "22pF" V 5112 825 50  0000 C CNN
@@
 AR Path="/5F1F1050/5F26BE32" Ref="C85"  Part="1"
 AR Path="/5F45D3C3/5F26BE32" Ref="C85"  Part="1"
+AR Path="/5F4B2714/5F26BE32" Ref="C?"  Part="1"
+AR Path="/5F4B67F1/5F26BE32" Ref="C?"  Part="1"
+AR Path="/5F4B8821/5F26BE32" Ref="C?"  Part="1"
 F 0 "C85" V 5021 1175 50  0000 C CNN
 F 1 "22pF" V 5112 1175 50  0000 C CNN
@@
 AR Path="/5F1F1050/5F1DC654" Ref="C90"  Part="1"
 AR Path="/5F45D3C3/5F1DC654" Ref="C91"  Part="1"
+AR Path="/5F4B2714/5F1DC654" Ref="C?"  Part="1"
+AR Path="/5F4B67F1/5F1DC654" Ref="C?"  Part="1"
+AR Path="/5F4B8821/5F1DC654" Ref="C?"  Part="1"
 F 0 "C91" V 3756 1900 50  0000 C CNN
 F 1 "0.1µF" V 3847 1900 50  0000 C CNN
@@
 AR Path="/5F1F1050/5F1E13AE" Ref="C86"  Part="1"
 AR Path="/5F45D3C3/5F1E13AE" Ref="C86"  Part="1"
+AR Path="/5F4B2714/5F1E13AE" Ref="C?"  Part="1"
+AR Path="/5F4B67F1/5F1E13AE" Ref="C?"  Part="1"
+AR Path="/5F4B8821/5F1E13AE" Ref="C?"  Part="1"
 F 0 "C86" V 3531 1275 50  0000 C CNN
 F 1 "0.1µF" V 3622 1275 50  0000 C CNN
@@
 AR Path="/5F1F1050/5F1E2915" Ref="C87"  Part="1"
 AR Path="/5F45D3C3/5F1E2915" Ref="C87"  Part="1"
+AR Path="/5F4B2714/5F1E2915" Ref="C?"  Part="1"
+AR Path="/5F4B67F1/5F1E2915" Ref="C?"  Part="1"
+AR Path="/5F4B8821/5F1E2915" Ref="C?"  Part="1"
 F 0 "C87" V 3781 1450 50  0000 C CNN
 F 1 "0.1µF" V 3872 1450 50  0000 C CNN
@@
 AR Path="/5F1F1050/5F1E4CF4" Ref="C88"  Part="1"
 AR Path="/5F45D3C3/5F1E4CF4" Ref="C89"  Part="1"
+AR Path="/5F4B2714/5F1E4CF4" Ref="C?"  Part="1"
+AR Path="/5F4B67F1/5F1E4CF4" Ref="C?"  Part="1"
+AR Path="/5F4B8821/5F1E4CF4" Ref="C?"  Part="1"
 F 0 "C89" V 3506 1725 50  0000 C CNN
 F 1 "0.1µF" V 3597 1725 50  0000 C CNN
@@
 AR Path="/5F1F1050/5F1DF03E" Ref="C?"  Part="1"
 AR Path="/5F45D3C3/5F1DF03E" Ref="C88"  Part="1"
+AR Path="/5F4B2714/5F1DF03E" Ref="C?"  Part="1"
+AR Path="/5F4B67F1/5F1DF03E" Ref="C?"  Part="1"
+AR Path="/5F4B8821/5F1DF03E" Ref="C?"  Part="1"
 F 0 "C88" V 5021 1475 50  0000 C CNN
 F 1 "22pF" V 5112 1475 50  0000 C CNN
@@
 USB data
 Text HLabel 5875 2825 0    50   Input ~ 0
-MOSI
+COPI
 Text HLabel 5875 2975 0    50   Input ~ 0
 SCK
-Text HLabel 5875 3125 0    50   Input ~ 0
-MISO
 NoConn ~ 6150 3275
 Wire Wire Line
@@
 AR Path="/5F1F1050/5F1F5B2A" Ref="U2"  Part="3"
 AR Path="/5F45D3C3/5F1F5B2A" Ref="U2"  Part="3"
+AR Path="/5F4B2714/5F1F5B2A" Ref="U?"  Part="3"
+AR Path="/5F4B67F1/5F1F5B2A" Ref="U?"  Part="3"
+AR Path="/5F4B8821/5F1F5B2A" Ref="U?"  Part="3"
 F 0 "U2" H 2775 3165 50  0000 C CNN
 F 1 "ATSAMD51J19A" H 2775 3074 50  0000 C CNN
@@
 AR Path="/5F1F1050/5F46DDBE" Ref="C?"  Part="1"
 AR Path="/5F45D3C3/5F46DDBE" Ref="C92"  Part="1"
+AR Path="/5F4B2714/5F46DDBE" Ref="C?"  Part="1"
+AR Path="/5F4B67F1/5F46DDBE" Ref="C?"  Part="1"
+AR Path="/5F4B8821/5F46DDBE" Ref="C?"  Part="1"
 F 0 "C92" H 1267 2921 50  0000 L CNN
 F 1 "0.1µF" H 1267 2830 50  0000 L CNN
@@
 AR Path="/5F1F1050/5F43F171" Ref="U?"  Part="1"
 AR Path="/5F45D3C3/5F43F171" Ref="U3"  Part="1"
+AR Path="/5F4B2714/5F43F171" Ref="U?"  Part="1"
+AR Path="/5F4B67F1/5F43F171" Ref="U?"  Part="1"
+AR Path="/5F4B8821/5F43F171" Ref="U?"  Part="1"
 F 0 "U3" H 2050 4997 50  0000 C CNN
 F 1 "S25FL064LABMFI013" H 2050 4906 50  0000 C CNN
@@
 AR Path="/5F1F1050/5F34C90C" Ref="R?"  Part="1"
 AR Path="/5F45D3C3/5F34C90C" Ref="R9"  Part="1"
+AR Path="/5F4B2714/5F34C90C" Ref="R?"  Part="1"
+AR Path="/5F4B67F1/5F34C90C" Ref="R?"  Part="1"
+AR Path="/5F4B8821/5F34C90C" Ref="R?"  Part="1"
 F 0 "R9" V 1155 3850 50  0000 C CNN
 F 1 "10k" V 1064 3850 50  0000 C CNN
@@
 AR Path="/5F1F1050/5F28C135" Ref="U2"  Part="2"
 AR Path="/5F45D3C3/5F28C135" Ref="U2"  Part="2"
+AR Path="/5F4B2714/5F28C135" Ref="U?"  Part="2"
+AR Path="/5F4B67F1/5F28C135" Ref="U?"  Part="2"
+AR Path="/5F4B8821/5F28C135" Ref="U?"  Part="2"
 F 0 "U2" H 2350 7865 50  0000 C CNN
 F 1 "ATSAMD51J19A" H 2350 7774 50  0000 C CNN
@@
 AR Path="/5F1F1050/5F2C4CD2" Ref="R8"  Part="1"
 AR Path="/5F45D3C3/5F2C4CD2" Ref="R8"  Part="1"
+AR Path="/5F4B2714/5F2C4CD2" Ref="R?"  Part="1"
+AR Path="/5F4B67F1/5F2C4CD2" Ref="R?"  Part="1"
+AR Path="/5F4B8821/5F2C4CD2" Ref="R?"  Part="1"
 F 0 "R8" V 10880 3075 50  0000 C CNN
 F 1 "10k" V 10789 3075 50  0000 C CNN
@@
 U 1 1 5F7FAE7A
 P 4200 3975
+AR Path="/5F45D3C3/5F7FAE7A" Ref="J2"  Part="1"
+AR Path="/5F4B2714/5F7FAE7A" Ref="J?"  Part="1"
+AR Path="/5F4B67F1/5F7FAE7A" Ref="J?"  Part="1"
+AR Path="/5F4B8821/5F7FAE7A" Ref="J?"  Part="1"
 F 0 "J2" V 3619 3975 50  0000 C CNN
 F 1 "SWD CONNECTOR" V 3710 3975 50  0000 C CNN
@@
 AR Path="/5F1F1050/5F264576" Ref="U2"  Part="1"
 AR Path="/5F45D3C3/5F264576" Ref="U2"  Part="1"
+AR Path="/5F4B2714/5F264576" Ref="U?"  Part="1"
+AR Path="/5F4B67F1/5F264576" Ref="U?"  Part="1"
+AR Path="/5F4B8821/5F264576" Ref="U?"  Part="1"
 F 0 "U2" H 8050 3490 50  0000 C CNN
 F 1 "ATSAMD51J19A" H 8050 3399 50  0000 C CNN
@@
 U 1 1 5F8C1CE8
 P 5225 4875
+AR Path="/5F45D3C3/5F8C1CE8" Ref="D?"  Part="1"
+AR Path="/5F4B2714/5F8C1CE8" Ref="D?"  Part="1"
+AR Path="/5F4B67F1/5F8C1CE8" Ref="D?"  Part="1"
+AR Path="/5F4B8821/5F8C1CE8" Ref="D?"  Part="1"
 F 0 "D?" H 5225 4670 50  0000 C CNN
 F 1 "LED_TX" H 5225 4761 50  0000 C CNN
@@
 U 1 1 5F8C3D21
 P 5225 5225
+AR Path="/5F45D3C3/5F8C3D21" Ref="D?"  Part="1"
+AR Path="/5F4B2714/5F8C3D21" Ref="D?"  Part="1"
+AR Path="/5F4B67F1/5F8C3D21" Ref="D?"  Part="1"
+AR Path="/5F4B8821/5F8C3D21" Ref="D?"  Part="1"
 F 0 "D?" H 5225 5020 50  0000 C CNN
 F 1 "LED_RX" H 5225 5111 50  0000 C CNN
@@
 U 1 1 5F8F99D2
 P 6000 4875
+AR Path="/5F45D3C3/5F8F99D2" Ref="R?"  Part="1"
+AR Path="/5F4B2714/5F8F99D2" Ref="R?"  Part="1"
+AR Path="/5F4B67F1/5F8F99D2" Ref="R?"  Part="1"
+AR Path="/5F4B8821/5F8F99D2" Ref="R?"  Part="1"
 F 0 "R?" V 5795 4875 50  0000 C CNN
 F 1 "1k" V 5886 4875 50  0000 C CNN
@@
 U 1 1 5F8FA351
 P 6000 5225
+AR Path="/5F45D3C3/5F8FA351" Ref="R?"  Part="1"
+AR Path="/5F4B2714/5F8FA351" Ref="R?"  Part="1"
+AR Path="/5F4B67F1/5F8FA351" Ref="R?"  Part="1"
+AR Path="/5F4B8821/5F8FA351" Ref="R?"  Part="1"
 F 0 "R?" V 5795 5225 50  0000 C CNN
 F 1 "1k" V 5886 5225 50  0000 C CNN
@@
 Text HLabel 10400 1125 2    50   Input ~ 0
 D13
+Text Notes 5575 6075 0    79   ~ 0
+heavily inspired by Adafruit M4 \nhttps://learn.adafruit.com/adafruit-metro-m4-express-featuring-atsamd51/downloads
+Text HLabel 5875 3125 0    50   Input ~ 0
+CIPO
 $EndSCHEMATC
