File: goLED.sch (KiCad schematic (older format))
At the start: 11 parts, among them J1 USB_C_Receptacle_USB2.0, U1 AP2112K-3.3

Commit message: update
Parts:
- added J?: Controller, symbol Connector:Conn_01x06_Male
- added J?: Digital I/O [0-9], symbol Connector:Conn_01x10_Male
- added J? (x2): Digital I/O [10-13], symbol Connector:Conn_01x04_Male
- added J?: Analog, symbol Connector:Conn_01x07_Male
- added J?: SPI, symbol Connector:Conn_01x03_Male
- added J?: I2C, symbol Connector:Conn_01x02_Male
Connections:
- net ATSAMD51/D10: now also J?.1 (Pin_1), J?.1 (Pin_1)
- net ATSAMD51/D11: now also J?.2 (Pin_2), J?.2 (Pin_2)
- net ATSAMD51/D12: now also J?.3 (Pin_3), J?.3 (Pin_3)
- net ATSAMD51/D13: now also J?.4 (Pin_4), J?.4 (Pin_4)
- new net ATSAMD51/A0: J?.1 (Pin_1)
- new net ATSAMD51/A1: J?.2 (Pin_2)
- new net ATSAMD51/A2: J?.3 (Pin_3)
- new net ATSAMD51/A3: J?.4 (Pin_4)
- new net ATSAMD51/A4: J?.5 (Pin_5)
- new net ATSAMD51/A5: J?.6 (Pin_6)
- new net ATSAMD51/AREF: J?.7 (Pin_7)
- new net ATSAMD51/CIPO: J?.2 (Pin_2)
- new net ATSAMD51/COPI: J?.3 (Pin_3)
- new net ATSAMD51/D0: J?.1 (Pin_1)
- new net ATSAMD51/D1: J?.2 (Pin_2)
- new net ATSAMD51/D2: J?.3 (Pin_3)
- new net ATSAMD51/D3: J?.4 (Pin_4)
- new net ATSAMD51/D4: J?.5 (Pin_5)
- new net ATSAMD51/D5: J?.6 (Pin_6)
- new net ATSAMD51/D6: J?.7 (Pin_7)
- new net ATSAMD51/D7: J?.8 (Pin_8)
- new net ATSAMD51/D8: J?.9 (Pin_9)
- new net ATSAMD51/D9: J?.10 (Pin_10)
- new net ATSAMD51/SCK: J?.1 (Pin_1)
- new net ATSAMD51/SCL: J?.1 (Pin_1)
- new net ATSAMD51/SDA: J?.2 (Pin_2)
- new net Controller/DIR: J?.3 (Pin_3)
- new net Controller/HORIZ_VERT: J?.4 (Pin_4)
- new net Controller/PASS_CONF: J?.2 (Pin_2)
- new net Controller/PLAYER: J?.5 (Pin_5)
- new net Controller/TRANSMITTING: J?.1 (Pin_1)
- new net Controller/VIN: J?.6 (Pin_6)
